Commit message: add MuJoCo model and SystemInterface

File: uav_description/urdf/quad.urdf.xacro (robot description, xacro)
@@ -2,11 +2,13 @@
 <robot name="quad_x" xmlns:xacro="http://ros.org/wiki/xacro">
   <xacro:include filename="rotor_link.xacro" />
-  <!--Skydio X2 configuration-->
-  <!--https://github.com/lvjonok/skydio_x2_description-->
   <link name="base_link" />
-  <xacro:rotor_link id="1" base="base_link" origin="-0.14 -0.18 0.05" radius="0.13" />
-  <xacro:rotor_link id="2" base="base_link" origin="-0.14 +0.18 0.05" radius="0.13" />
-  <xacro:rotor_link id="3" base="base_link" origin="+0.14 +0.18 0.08" radius="0.13" />
-  <xacro:rotor_link id="4" base="base_link" origin="+0.14 -0.18 0.08" radius="0.13" />
+  <!--ZMR 250 frame-->
+  <xacro:property name="W" value="0.210"/>
+  <xacro:property name="H" value="0.155"/>
+  <!--rotation direction: 1: CCW, 2: CW, 3: CCW, 4: CW-->
+  <xacro:rotor_link id="1" base="base_link" origin="+${H/2} -${W/2} 0" radius="0.07" />
+  <xacro:rotor_link id="2" base="base_link" origin="+${H/2} +${W/2} 0" radius="0.07" />
+  <xacro:rotor_link id="3" base="base_link" origin="-${H/2} +${W/2} 0" radius="0.07" />
+  <xacro:rotor_link id="4" base="base_link" origin="-${H/2} -${W/2} 0" radius="0.07" />
   <link name="base_imu" />
   <joint name="base_imu_joint" type="fixed">
@@ -14,5 +16,5 @@
     <child link="base_imu" />
   </joint>
-  <xacro:include filename="$(find uav_description)/urdf/ros2_control/proxy_interfaces.xacro" />
-  <xacro:proxy_interfaces />
+  <xacro:include filename="$(find uav_description)/urdf/ros2_control/mujoco_interface.xacro" />
+  <xacro:mujoco_interface />
 </robot>

Commit message: define rotor inertia

File: uav_description/urdf/quad.urdf.xacro (robot description, xacro)
@@ -7,8 +7,8 @@
   <xacro:property name="H" value="0.155"/>
   <!--rotation direction: 1: CCW, 2: CW, 3: CCW, 4: CW-->
-  <xacro:rotor_link id="1" base="base_link" origin="+${H/2} -${W/2} 0" radius="0.07" />
-  <xacro:rotor_link id="2" base="base_link" origin="+${H/2} +${W/2} 0" radius="0.07" />
-  <xacro:rotor_link id="3" base="base_link" origin="-${H/2} +${W/2} 0" radius="0.07" />
-  <xacro:rotor_link id="4" base="base_link" origin="-${H/2} -${W/2} 0" radius="0.07" />
+  <xacro:rotor_link id="1" base="base_link" origin="+${H/2} -${W/2} 0" radius="0.07"/>
+  <xacro:rotor_link id="2" base="base_link" origin="+${H/2} +${W/2} 0" radius="0.07"/>
+  <xacro:rotor_link id="3" base="base_link" origin="-${H/2} +${W/2} 0" radius="0.07"/>
+  <xacro:rotor_link id="4" base="base_link" origin="-${H/2} -${W/2} 0" radius="0.07"/>
   <link name="base_imu" />
   <joint name="base_imu_joint" type="fixed">

File: uav_description/urdf/rotor_link.xacro (robot description, xacro)
@@ -1,9 +1,19 @@
 <?xml version="1.0"?>
 <robot name="rotor_link" xmlns:xacro="http://ros.org/wiki/xacro">
-  <xacro:macro name="rotor_link" params="id base origin radius">
+  <xacro:macro name="rotor_link" params="id base origin radius mass=0.01">
+    <xacro:property name="width" value="0.001" />
     <link name="rotor/${id}">
+      <inertial>
+        <mass value="${mass}"/>
+        <inertia
+          ixx="${(1/4*mass*radius*radius + 1/12*mass*width*width)}"
+          iyy="${(1/4*mass*radius*radius + 1/12*mass*width*width)}"
+          izz="${(1/2*mass*radius*radius)}"
+          ixy="0" ixz="0" iyz="0"
+        />
+      </inertial>
       <visual>
         <geometry>
-          <cylinder radius="${radius}" length="0.001" />
+          <cylinder radius="${radius}" length="${width}" />
         </geometry>
       </visual>

Commit message: single URDF with switch for types

File: uav_description/urdf/quad.urdf.xacro (robot description, xacro)
@@ -1,6 +1,17 @@
 <?xml version="1.0"?>
-<robot name="quad_x" xmlns:xacro="http://ros.org/wiki/xacro" version="1.1">
+<robot name="quad" xmlns:xacro="http://ros.org/wiki/xacro" version="1.1">
+  <xacro:arg name="model" default="proxy"/>
+  <xacro:property name="model" value="$(arg model)"/>
+  <xacro:if value="${model == 'pifly'}">
+    <xacro:arg name="imu_quat" default="0 0 1 0"/>
+  </xacro:if>
   <xacro:include filename="zmr250.urdf.xacro" />
   <xacro:include filename="$(find uav_description)/urdf/ros2_control/proxy.ros2_control.xacro" />
-  <xacro:proxy_ros2_control />
+  <xacro:include filename="$(find uav_description)/urdf/ros2_control/pifly.ros2_control.xacro" />
+  <xacro:if value="${model == 'proxy'}">
+    <xacro:proxy_ros2_control />
+  </xacro:if>
+  <xacro:if value="${model == 'pifly'}">
+    <xacro:pifly_ros2_control />
+  </xacro:if>
 </robot>
