Commit message: base ZMR 250 URDF with 'proxy' and 'pifly' ros2_control macros

File: uav_description/urdf/pifly.urdf.xacro (robot description, xacro)
@@ -1,63 +1,7 @@
 <?xml version="1.0"?>
-<robot name="pifly" xmlns:xacro="http://ros.org/wiki/xacro">
-  <xacro:include filename="rotor_link.xacro" />
-  <link name="base_link" />
-  <!--ZMR 250 frame-->
-  <xacro:property name="W" value="0.210"/>
-  <xacro:property name="H" value="0.155"/>
-  <!--rotation direction: 1: CCW, 2: CW, 3: CCW, 4: CW-->
-  <xacro:rotor_link id="1" base="base_link" origin="+${H/2} -${W/2} 0" radius="0.07" />
-  <xacro:rotor_link id="2" base="base_link" origin="+${H/2} +${W/2} 0" radius="0.07" />
-  <xacro:rotor_link id="3" base="base_link" origin="-${H/2} +${W/2} 0" radius="0.07" />
-  <xacro:rotor_link id="4" base="base_link" origin="-${H/2} -${W/2} 0" radius="0.07" />
-  <link name="base_imu" />
-  <joint name="base_imu_joint" type="fixed">
-    <parent link="base_link" />
-    <child link="base_imu" />
-    <origin rpy="0 0 ${pi}" />
-  </joint>
-  <xacro:include filename="$(find uav_description)/urdf/interfaces/imu_interface.xacro" />
-  <xacro:include filename="$(find uav_description)/urdf/interfaces/magnetometer_interface.xacro" />
-  <xacro:include filename="$(find uav_description)/urdf/interfaces/rotor_interface.xacro" />
-  <xacro:include filename="$(find uav_description)/urdf/interfaces/rc_interface.xacro" />
-  <xacro:macro name="rotors">
-    <xacro:rotor id="1" />
-    <xacro:rotor id="2" />
-    <xacro:rotor id="3" />
-    <xacro:rotor id="4" />
-  </xacro:macro>
-  <ros2_control name="imu" type="sensor">
-    <properties>
-      <async thread_priority="90"/>
-    </properties>
-    <hardware>
-      <plugin>uav/drivers/MPU9250</plugin>
-      <param name="sensor_name">base_imu</param>
-      <param name="bus">1</param>
-      <param name="calibration_file">$(find uav_description)/calibration/pifly.yaml</param>
-    </hardware>
-    <xacro:imu name="base_imu" />
-    <xacro:magnetometer name="base_imu" />
-  </ros2_control>
-  <ros2_control name="pwm" type="actuator" is_async="true" rw_rate="400">
-    <properties>
-      <async thread_priority="90"/>
-    </properties>
-    <hardware>
-      <plugin>uav/drivers/PCA9685</plugin>
-      <param name="bus">1</param>
-    </hardware>
-    <xacro:rotors />
-  </ros2_control>
-  <!-- FrSky S.BUS frame is transmitted every 9 ms -->
-  <ros2_control name="rc" type="sensor" is_async="true" rw_rate="100">
-    <properties>
-      <async thread_priority="90"/>
-    </properties>
-    <hardware>
-      <plugin>uav/drivers/SBUS</plugin>
-      <param name="device">/dev/ttyAMA0</param>
-    </hardware>
-    <xacro:rc />
-  </ros2_control>
+<robot name="pifly" xmlns:xacro="http://ros.org/wiki/xacro" version="1.1">
+  <xacro:arg name="imu_quat" default="0 0 1 0"/>
+  <xacro:include filename="zmr250.urdf.xacro" />
+  <xacro:include filename="$(find uav_description)/urdf/ros2_control/pifly.ros2_control.xacro" />
+  <xacro:pifly_ros2_control />
 </robot>

File: uav_description/urdf/quad.urdf.xacro (robot description, xacro)
@@ -1,18 +1,6 @@
 <?xml version="1.0"?>
-<robot name="quad_x" xmlns:xacro="http://ros.org/wiki/xacro">
-  <xacro:include filename="rotor_link.xacro" />
-  <!--Skydio X2 configuration-->
-  <!--https://github.com/lvjonok/skydio_x2_description-->
-  <link name="base_link" />
-  <xacro:rotor_link id="1" base="base_link" origin="-0.14 -0.18 0.05" radius="0.13" />
-  <xacro:rotor_link id="2" base="base_link" origin="-0.14 +0.18 0.05" radius="0.13" />
-  <xacro:rotor_link id="3" base="base_link" origin="+0.14 +0.18 0.08" radius="0.13" />
-  <xacro:rotor_link id="4" base="base_link" origin="+0.14 -0.18 0.08" radius="0.13" />
-  <link name="base_imu" />
-  <joint name="base_imu_joint" type="fixed">
-    <parent link="base_link" />
-    <child link="base_imu" />
-  </joint>
-  <xacro:include filename="$(find uav_description)/urdf/ros2_control/proxy_interfaces.xacro" />
-  <xacro:proxy_interfaces />
+<robot name="quad_x" xmlns:xacro="http://ros.org/wiki/xacro" version="1.1">
+  <xacro:include filename="zmr250.urdf.xacro" />
+  <xacro:include filename="$(find uav_description)/urdf/ros2_control/proxy.ros2_control.xacro" />
+  <xacro:proxy_ros2_control />
 </robot>

File: uav_description/urdf/ros2_control/proxy.ros2_control.xacro (robot description, xacro)
@@ -1,5 +1,5 @@
 <?xml version="1.0"?>
-<robot name="proxy" xmlns:xacro="http://ros.org/wiki/xacro">
-  <xacro:macro name="proxy_interfaces">
+<robot xmlns:xacro="http://ros.org/wiki/xacro">
+  <xacro:macro name="proxy_ros2_control">
     <xacro:include filename="$(find uav_description)/urdf/interfaces/imu_interface.xacro" />
     <xacro:include filename="$(find uav_description)/urdf/interfaces/rotor_interface.xacro" />
